File: PCBs/Mainboard/bic.kicad_sch (KiCad schematic)
At the start: 19 parts, among them IC4 MIC5303-1.8YMT-TR, J2 TERMISTOR, J3 BAT_CONN, U2 BQ25628ERYKR, U3 TPS62291DRVR

Commit message: Fix schematic title
Also update to KiCAD 9
Changed lines of the file:
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@@
 (kicad_sch
-	(version 20231120)
+	(version 20250114)
 	(generator "eeschema")
-	(generator_version "8.0")
+	(generator_version "9.0")
 	(paper "A4")
 	(title_block
