File: PCBs/Mainboard/display.kicad_sch (KiCad schematic)
At the start: 9 parts, among them J5 Conn_02x12_Counter_Clockwise_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, U4 TPS65136RTER

Commit message: Fix schematic title
Also update to KiCAD 9
Changed lines of the file:
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@@
 (kicad_sch
-	(version 20231120)
+	(version 20250114)
 	(generator "eeschema")
-	(generator_version "8.0")
+	(generator_version "9.0")
 	(paper "A4")
 	(title_block
