File: PCBs/Mainboard/imu.kicad_sch (KiCad schematic)
At the start: 4 parts, among them IC1 ICM-42670-P

Commit message: Fix schematic title
Also update to KiCAD 9
Other:
- title: Battery IC & Step-down -> IMU
Changed lines of the file:
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@@
 (kicad_sch
-	(version 20231120)
+	(version 20250114)
 	(generator "eeschema")
-	(generator_version "8.0")
+	(generator_version "9.0")
 	(paper "A4")
 	(title_block
-		(title "Battery IC & Step-down")
+		(title "IMU")
 	)
 	(junction
