File: PCBs/Mainboard/nfc.kicad_sch (KiCad schematic)
At the start: 35 parts, among them IC2 ST25R3916-AQET, J4 NFC_ANTENNA, Y2 27.12MHz

Commit message: Fix schematic title
Also update to KiCAD 9
Changed lines of the file:
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@@
 (kicad_sch
-	(version 20231120)
+	(version 20250114)
 	(generator "eeschema")
-	(generator_version "8.0")
+	(generator_version "9.0")
 	(paper "A4")
 	(title_block
