File: PCBs/plajtime-main/plajtime-main.kicad_pcb (KiCad board)
At the start: 4 copper layers, 31.2 x 34 mm, 82 parts, among them J1 RP SWD, J2 Internal connector, J3 Display connector, J4 Extention connector, J5 Battery connector, J6 Nordic SWD, J7 NFC connector, U1 W25Q64JWU, U2 MP2664, U3 TPS63031DSK, U4 RP2350A, U5 BMA456, U6 MAX17055, U7 RV-3028-C7, U8 nRF52833_QDxx, U9 W25Q64JWU, Y1 13MHz, Y2 32MHz

Commit message: Some layout is done
Parts:
- removed AE1: Antenna_Chip, RF_Antenna:Johanson_2450AT18x100_2400-2500Mhz
- removed C17, C20: 10uF, Capacitor_SMD:C_0402_1005Metric
- added C47: 0.1uF, Capacitor_SMD:C_0201_0603Metric, B.Cu at (41.6, 148.6)
- added J8: Battery Connector, Library:CONN_505066-0622_MOL, F.Cu at (37.1, 138.3)
- added R12: 133k, Resistor_SMD:R_0201_0603Metric, B.Cu at (38.5, 141.4)
- C1, C12, C14, C16, C18, C19, C21, C22, C24, C26, C29, C30, C31, C32, C33, C37, C38, C4, C41, C42, C44, C8, L5, L6, R1, R11, R4, R5, R6, R7, R8, R9: moved to B.Cu
- C5: value 0.1uF -> 4.7uF; footprint Capacitor_SMD:C_0201_0603Metric -> Capacitor_SMD:C_0402_1005Metric; moved to B.Cu
- J1: footprint Connector_PinHeader_1.00mm:PinHeader_1x03_P1.00mm_Vertical -> Library:PinHeader_1x03_P1.00mm_Vertical
- J4: footprint Library:FPC_7 -> Library:5050660822
- J5: value Battery connector -> Conn_Coaxial; footprint Library:CONN8_505004-0812_MOL -> Library:W.FL_Hirose_W.FL2-R-SMT-1_Vertical
- J6: footprint Connector_PinHeader_1.00mm:PinHeader_1x03_P1.00mm_Vertical -> Library:PinHeader_1x03_P1.00mm_Vertical; moved to B.Cu
- J7: value NFC connector -> Conn_Coaxial; footprint Library:FPC_4 -> Library:W.FL_Hirose_W.FL2-R-SMT-1_Vertical
- L1: value 1.5uH -> 1uH
- U1: value W25Q64JWU -> W25Q64JWBYIM; footprint Package_CSP:WLCSP-8_1.551x2.284mm_Layout2x4_P0.5mm -> Library:BGA-24_4x6_6.0x6.0mm; moved to B.Cu
- U3: value TPS63031DSK -> TPS628438YKA; footprint Package_SON:WSON-10-1EP_2.5x2.5mm_P0.5mm_EP1.2x2mm -> Package_BGA:Texas_DSBGA-6_0.757x1.01mm_Layout2x3_P0.35mm; moved to B.Cu
- U9: moved to F.Cu
- moved R4 66.1 mm to (37.0, 133.8), turned to 45 degrees
- moved L6 60.8 mm to (45.3, 146.5), turned to 90 degrees
- moved C37 57.6 mm to (43.3, 145.2), turned to -90 degrees
- moved C38 57.5 mm to (42.4, 145.2), turned to -90 degrees
- moved C15 57.5 mm to (38.6, 141.3)
- moved C1 57.4 mm to (37.0, 143.8)
- moved C18 55.2 mm to (38.8, 139.5), turned to -135 degrees
- moved R6 54.8 mm to (39.1, 146.7), turned to 180 degrees
- moved C33 53.5 mm to (41.5, 146.0), turned to -90 degrees
- moved C44 53.4 mm to (46.9, 147.0), turned to -90 degrees
- moved C46 52.7 mm to (40.6, 152.1), turned to -135 degrees
- moved C45 52.3 mm to (41.6, 151.0), turned to 75 degrees
- moved C43 50.6 mm to (45.6, 151.4), turned to -90 degrees
- moved C30 50.3 mm to (39.1, 145.8), turned to 180 degrees
- moved L3 50.2 mm to (43.7, 153.8), turned to 90 degrees
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Connections:
- C1 pad 1: VSYS -> +3V
- C38 pad 1: +3.3V -> +5V
- C45 pad 1: Net-(J7-Pin_1) -> Net-(J7-In)
- C46 pad 1: Net-(J7-Pin_3) -> Net-(J7-Ext)
- C5 pad 1: Net-(U3-EN) -> VSYS
- J2 pad 4: RP_SDA -> RP_SCL
- J2 pad 5: RP_SCL -> RP_SDA
- J3 pad 29: VSYS -> +3.3V
- J3 pad 30: VSYS -> +3.3V
- J4 pad 2: SDA -> SCL
- J4 pad 3: SCL -> /EXT_INT
- J4 pad 4: /EXT_INT -> SDA
- J4 pad 6: /EXT_GPIO -> unconnected-(J4-Pin_6-Pad6)
- J4 pad 7: GND -> /EXT_GPIO
- J4 pad MP: unconnected-(J4-MountPin-PadMP) -> GND
- J5 pad 1: +BATT -> Net-(J5-In)
- J5 pad 2: unconnected-(J5-Pin_2-Pad2) -> GND
- J7 pad 1: Net-(J7-Pin_1) -> Net-(J7-In)
- J7 pad 2: Net-(J7-Pin_1) -> Net-(J7-Ext)
- L1 pad 1: Net-(U3-L2) -> Net-(U3-SW)
- L1 pad 2: Net-(U3-L1) -> +3V
- L3 pad 1: Net-(AE1-PCB_Trace) -> Net-(J5-In)
- U1 pad B2: (no net) -> +3.3V
- U1 pad C2: (no net) -> /QMI_SD3
- U1 pad D2: (no net) -> /QMI_SCLK
- U4 pad 14: /DISP_SCL -> /DISP_RST
- U4 pad 15: /DISP_DIO0 -> /DISP_CS
- U4 pad 16: /DISP_DI1 -> /DISP_DIO0
- U4 pad 17: /DISP_DI2 -> /DISP_DI1
- U4 pad 18: /DISP_DI3 -> /DISP_DI2
- U4 pad 19: /DISP_CS -> /DISP_DI3
- U4 pad 26: unconnected-(U4-RUN-Pad26) -> +3.3V
- U4 pad 27: /DISP_RST -> /TP_INT
- U4 pad 28: /TP_RESET -> /DISP_SCL
- U4 pad 29: /DISP_TE -> /TP_RESET
- U4 pad 32: /TP_INT -> unconnected-(U4-GPIO20-Pad32)
- U4 pad 33: /VIC_INT -> unconnected-(U4-GPIO21-Pad33)
- U4 pad 34: /SLIDER_INT -> UART_TX
- U4 pad 35: /CLK_OUT -> UART_RX
- U4 pad 36: unconnected-(U4-GPIO24-Pad36) -> /SLIDER_INT
- U4 pad 37: unconnected-(U4-GPIO25-Pad37) -> /CLK_OUT
- U4 pad 5: unconnected-(U4-GPIO3-Pad5) -> /DISP_TE
- U4 pad 60: /QMI_CS1 -> /QMI_CS0
- U6 pad 11: -BATT -> unconnected-(U6-CSP-Pad11)
- U8 pad 10: +3.3V -> +5V
- U8 pad 19: Net-(J6-Pin_2) -> Net-(J6-Pin_3)
- U8 pad 2: unconnected-(U8-XL1/P0.00-Pad2) -> SDA
- U8 pad 20: Net-(J6-Pin_3) -> Net-(J6-Pin_2)
- U8 pad 22: Net-(J7-Pin_1) -> Net-(J7-In)
- U8 pad 23: Net-(J7-Pin_3) -> Net-(J7-Ext)
- U8 pad 3: unconnected-(U8-XL2/P0.01-Pad3) -> SCL
- U8 pad 4: SDA -> unconnected-(U8-AIN2/P0.04-Pad4)
- U8 pad 5: SCL -> unconnected-(U8-AIN3/P0.05-Pad5)
Routing:
- net /TP_INT: track 0.00 -> 21.5 mm, vias 0 -> 2
- net /TP_RESET: track 0.00 -> 20.7 mm, vias 0 -> 2
- net /DISP_EN: track 0.00 -> 19.7 mm, vias 0 -> 3
- net /DISP_SCL: track 1.14 -> 20.1 mm, vias 1 -> 2
- net +3.3V: track 7.39 -> 23.2 mm, vias 3 -> 19
- net RP_SCL: track 0.00 -> 15.5 mm, vias 0 -> 2
- net /DISP_DI3: track 1.01 -> 15.4 mm, vias 1 -> 2
- net RP_SDA: track 0.00 -> 14.0 mm, vias 0 -> 2
- net /DISP_DI2: track 0.88 -> 14.4 mm, vias 1 -> 0
- net /DISP_CS: track 1.13 -> 13.6 mm, vias 1 -> 2
- net /DISP_DI1: track 0.92 -> 13.2 mm, vias 1 -> 0
- net /DISP_RST: track 0.00 -> 11.9 mm, vias 0 -> 2
- net /DISP_DIO0: track 0.88 -> 11.7 mm, vias 1 -> 0
- net GND: track 0.98 -> 11.6 mm, vias 0 -> 28
- net -BATT: track 0.00 -> 9.10 mm, vias 0 -> 2
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- added copper zone on In3.Cu, net GND
- added copper zone on In4.Cu, net GND
Other:
- board size 31.2 x 34 mm -> 15.2 x 34 mm
- copper layers 4 -> 6

Commit message: Final?
Parts:
- added J9: RP USB, Library:PinHeader_1x03_P1.00mm_Vertical, B.Cu at (44.0, 131.8)
- U3: footprint Package_BGA:Texas_DSBGA-6_0.757x1.01mm_Layout2x3_P0.35mm -> Library:Texas_DSBGA-6_0.757x1.01mm_Layout2x3_P0.35mm
- moved J1 3.44 mm to (48.4, 127.5), turned to 45 degrees
- moved R6 2.52 mm to (37.5, 144.8), turned to 0 degrees
- moved R5 2.40 mm to (37.6, 146.7), turned to 0 degrees
- moved J6 2.08 mm to (39.9, 147.6), turned to 110 degrees
- moved C30 1.54 mm to (37.6, 145.8)
- moved C29 1.27 mm to (39.6, 142.6), turned to 90 degrees
- moved C33 1.22 mm to (41.5, 144.8), turned to 90 degrees
- moved C22 1.09 mm to (41.8, 126.5), turned to 45 degrees
- moved U7 1.05 mm to (38.0, 145.4), turned to 180 degrees
- moved C24 0.93 mm to (41.1, 143.5), turned to 180 degrees
- moved J8 0.39 mm to (37.1, 138.7)
- moved C26 0.39 mm to (36.5, 135.9)
- moved C28 0.39 mm to (36.5, 135.9)
- moved R4 0.39 mm to (37.0, 134.2)
- moved U6 0.39 mm to (38.2, 134.4)
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Connections:
- C12 pad 1: +3.3V -> +3V
- C14 pad 1: +3.3V -> +3V
- C16 pad 1: +3.3V -> +3V
- C19 pad 1: +3.3V -> +3V
- C21 pad 1: +3.3V -> +3V
- C22 pad 1: +3.3V -> +3V
- C23 pad 1: +3.3V -> +3V
- C24 pad 1: +3.3V -> +3V
- C25 pad 1: +3.3V -> +3V
- C27 pad 1: +3.3V -> +3V
- C29 pad 1: +3.3V -> +3V
- C3 pad 1: +3.3V -> +3V
- C30 pad 2: +3.3V -> +3V
- C31 pad 1: +3.3V -> +3V
- C32 pad 1: +3.3V -> +3V
- C33 pad 1: +3.3V -> +3V
- C37 pad 1: +3.3V -> +3V
- C47 pad 1: +3.3V -> +3V
- J2 pad 2: SDA -> SCL
- J2 pad 3: SCL -> SDA
- J3 pad 11: +3.3V -> +3V
- J3 pad 23: +3.3V -> +3V
- J3 pad 25: +3.3V -> +3V
- J3 pad 29: +3.3V -> +3V
- J3 pad 30: +3.3V -> +3V
- J4 pad 1: +3.3V -> +3V
- J4 pad 2: SCL -> /EXT_INT
- J4 pad 3: /EXT_INT -> /EXT_GPIO_2
- J4 pad 4: SDA -> /EXT_RST
- J4 pad 5: /EXT_RST -> SDA
- J4 pad 6: unconnected-(J4-Pin_6-Pad6) -> /EXT_GPIO_1
- J4 pad 7: /EXT_GPIO -> SCL
- J6 pad 1: GND -> Net-(J6-Pin_1)
- R10 pad 1: +3.3V -> +3V
- R2 pad 1: +3.3V -> +3V
- R7 pad 1: +3.3V -> +3V
- R8 pad 1: +3.3V -> +3V
- R9 pad 1: +3.3V -> +3V
- U1 pad B2: +3.3V -> +3V
- U4 pad 1: +3.3V -> +3V
- U4 pad 11: +3.3V -> +3V
- U4 pad 20: +3.3V -> +3V
- U4 pad 24: Net-(J1-Pin_3) -> Net-(J1-Pin_2)
- U4 pad 25: Net-(J1-Pin_2) -> Net-(J1-Pin_3)
- U4 pad 26: +3.3V -> +3V
- U4 pad 3: unconnected-(U4-GPIO1-Pad3) -> /SLIDER_INT
- U4 pad 30: +3.3V -> +3V
- U4 pad 32: unconnected-(U4-GPIO20-Pad32) -> /VIC_INT
- U4 pad 36: /SLIDER_INT -> unconnected-(U4-GPIO24-Pad36)
- U4 pad 38: +3.3V -> +3V
- U4 pad 44: +3.3V -> +3V
- U4 pad 45: +3.3V -> +3V
- U4 pad 49: +3.3V -> +3V
- U4 pad 51: unconnected-(U4-USB_DM-Pad51) -> Net-(J9-Pin_3)
- U4 pad 52: unconnected-(U4-USB_DP-Pad52) -> Net-(J9-Pin_2)
- U4 pad 53: +3.3V -> +3V
- U4 pad 54: +3.3V -> +3V
- U5 pad 10: +3.3V -> +3V
- U5 pad 3: +3.3V -> +3V
- U5 pad 7: +3.3V -> +3V
- U6 pad 11: unconnected-(U6-CSP-Pad11) -> -BATT
- U7 pad 7: +3.3V -> +3V
- U8 pad 11: +3.3V -> +3V
- U8 pad 16: Net-(U8-P0.18/~{RESET}) -> Net-(J6-Pin_1)
- U8 pad 17: GPU_INT -> /RTC_INT
- U8 pad 18: +3.3V -> +3V
- U8 pad 19: Net-(J6-Pin_3) -> Net-(J6-Pin_2)
- U8 pad 20: Net-(J6-Pin_2) -> Net-(J6-Pin_3)
- U8 pad 30: +3.3V -> +3V
- U8 pad 31: /IMU_INT_2 -> /IMU_INT_1
- U8 pad 32: /IMU_INT_1 -> /IMU_INT_2
- U8 pad 33: /CHARGER_INT -> /EXT_GPIO_2
- U8 pad 36: /GAUGE_INT -> /EXT_GPIO_1
- U8 pad 4: unconnected-(U8-AIN2/P0.04-Pad4) -> GPU_INT
- U8 pad 40: +3.3V -> +3V
- U8 pad 5: unconnected-(U8-AIN3/P0.05-Pad5) -> /GAUGE_INT
- U8 pad 6: /RTC_INT -> /OXY_INT
- U8 pad 7: /OXY_INT -> /CHARGER_INT
- U8 pad 8: +3.3V -> +3V
- U8 pad 9: +3.3V -> +3V
- U9 pad 8: +3.3V -> +3V
Routing:
- net SDA: track 0.00 -> 35.4 mm, vias 0 -> 6
- net SCL: track 0.00 -> 32.3 mm, vias 0 -> 6
- net UART_TX: track 0.00 -> 30.4 mm, vias 0 -> 2
- net UART_RX: track 0.00 -> 28.9 mm, vias 0 -> 2
- net /CLK_OUT: track 0.00 -> 27.3 mm, vias 0 -> 2
- net +3V: track 1.80 -> 27.6 mm, vias 1 -> 25
- net +3.3V: track 23.2 -> 0.00 mm, vias 19 -> 0
- net /VIC_INT: track 0.00 -> 19.0 mm, vias 0 -> 2
- net /GAUGE_INT: track 0.00 -> 15.1 mm
- net /IMU_INT_2: track 0.00 -> 12.5 mm, vias 0 -> 2
- net /IMU_INT_1: track 0.00 -> 12.4 mm, vias 0 -> 2
- net USB_D-: track 0.00 -> 12.2 mm, vias 0 -> 2
- net GPU_INT: track 0.00 -> 12.1 mm, vias 0 -> 2
- net GND: track 11.6 -> 23.2 mm, vias 28 -> 80
- net USB_D+: track 0.00 -> 10.7 mm, vias 0 -> 2
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- added copper zone on F.Cu, net +1V1
- added copper zone on In2.Cu, net +3V
- removed copper zone on In2.Cu, net +3.3V

Commit message: Some small changes
Routing:
- net +1V1: track 14.7 -> 15.8 mm
- net +3V: track 27.6 -> 27.0 mm
- net GND: track 23.2 -> 22.9 mm, vias 80 -> 83
Other:
- board text added: "<USB"
- board text added: "Plajtime v0.4 Mainboard"
- board text added: "RP SWD"
- board text added: "Smrt1"
- board text added: "Smrt2"
- board text added: "by Plajta"
- board text added: "nRF SWD"

Commit message: Add and modify labels
Modify mainly text thickness
Other:
- board text added: "AUX"
- board text added: "BAT"
- board text added: "Display"
- board text added: "EXP"
- board text added: "RF magic"
Changed lines of the file:
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@@
 		(layer "User.4")
+	)
+	(gr_text "Display"
+		(at 50 135.4 90)
+		(layer "F.SilkS")
+		(effects
+			(font
+				(size 0.6 0.6)
+				(thickness 0.1)
+				(bold yes)
+			)
+			(justify left bottom)
+		)
+	)
+	(gr_text "AUX"
+		(at 46 142 90)
+		(layer "F.SilkS")
+		(effects
+			(font
+				(size 0.6 0.6)
+				(thickness 0.1)
+				(bold yes)
+			)
+			(justify left bottom)
+		)
+	)
+	(gr_text "RF\nmagic"
+		(at 43.4 152.4 45)
+		(layer "F.SilkS")
+		(effects
+			(font
+				(size 0.5 0.5)
+				(thickness 0.1)
+			)
+			(justify right bottom)
+		)
+	)
+	(gr_text "EXP"
+		(at 47.8 145 0)
+		(layer "F.SilkS")
+		(effects
+			(font
+				(size 0.6 0.6)
+				(thickness 0.1)
+				(bold yes)
+			)
+			(justify left bottom)
+		)
+	)
+	(gr_text "BAT"
+		(at 39.4 138.4 90)
+		(layer "F.SilkS")
+		(effects
+			(font
+				(size 0.6 0.6)
+				(thickness 0.1)
+				(bold yes)
+			)
+			(justify left bottom)
+		)
 	)
 	(gr_text "by Plajta"
@@
 			(font
 				(size 0.8 0.8)
-				(thickness 0.1)
+				(thickness 0.15)
+				(bold yes)
 			)
 			(justify left bottom mirror)

Commit message: Move text around a bit
for future fruity changes
Other:
- board text added: "2nd flash/RAM"
- board text added: "Plajtime v0.4"
- board text added: "RP USB"
- board text added: "SMRT1"
- board text added: "SMRT2 ->"
- board text removed: "<USB"
- board text removed: "Plajtime v0.4 Mainboard"
- board text removed: "Smrt1"
- board text removed: "Smrt2"
Changed lines of the file:
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@@
 		)
 	)
-	(gr_text "Plajtime v0.4\nMainboard"
+	(gr_text "Plajtime\nv0.4"
 		(at 47.07 131.94 315)
 		(layer "B.SilkS")
@@
 		)
 	)
-	(gr_text "Smrt1"
-		(at 43.459611 135.463099 315)
+	(gr_text "SMRT1"
+		(at 43.6 135.7 315)
 		(layer "B.SilkS")
 		(effects
@@
 	)
 	(gr_text "nRF SWD"
-		(at 41.25 147.82 45)
+		(at 41.2 151 315)
 		(layer "B.SilkS")
 		(effects
@@
 		)
 	)
-	(gr_text "Smrt2"
-		(at 38.07 140.76 0)
+	(gr_text "SMRT2 ->"
+		(at 37.4 136.8 90)
 		(layer "B.SilkS")
 		(effects
@@
 		)
 	)
-	(gr_text "<USB"
-		(at 41.92 130.13 315)
+	(gr_text "RP USB"
+		(at 47.1 133.5 345)
 		(layer "B.SilkS")
 		(effects
@@
 		)
 	)
+	(gr_text "2nd flash/RAM"
+		(at 42.4 133.3 45)
+		(layer "B.SilkS")
+		(effects
+			(font
+				(size 0.5 0.5)
+				(thickness 0.1)
+			)
+			(justify left bottom mirror)
+		)
+	)
+	(dimension
+		(type orthogonal)
+		(layer "Cmts.User")
+		(pts
+			(xy 50.42 139.579998) (xy 35.22 139.579998)
+		)
+		(height -20.179998)
+		(orientation 0)
+		(format
+			(prefix "")
+			(suffix "")
+			(units 3)
+			(units_format 0)
+			(precision 4)
+			(suppress_zeroes yes)
+		)
+		(style
+			(thickness 0.1)
+			(arrow_length 1.27)
+			(text_position_mode 0)
+			(arrow_direction outward)
+			(extension_height 0.58642)
+			(extension_offset 0.5)
+			(keep_text_aligned yes)
+		)
+		(gr_text "15,2"
+			(at 42.82 118.25 0)
+			(layer "Cmts.User")
+			(effects
+				(font
+					(size 1 1)
+					(thickness 0.15)
+				)
+			)
+		)
+	)
+	(dimension
+		(type orthogonal)
+		(layer "Cmts.User")
+		(pts
+			(xy 49.42 156.58) (xy 49.42 122.579998)
+		)
+		(height 5.78)
+		(orientation 1)
+		(format
+			(prefix "")
+			(suffix "")
+			(units 3)
+			(units_format 0)
+			(precision 4)
+			(suppress_zeroes yes)
+		)
+		(style
+			(thickness 0.1)
+			(arrow_length 1.27)
+			(text_position_mode 0)
+			(arrow_direction outward)
+			(extension_height 0.58642)
+			(extension_offset 0.5)
+			(keep_text_aligned yes)
+		)
+		(gr_text "34"
+			(at 54.05 139.579999 90)
+			(layer "Cmts.User")
+			(effects
+				(font
+					(size 1 1)
+					(thickness 0.15)
+				)
+			)
+		)
+	)

Commit message: Add a nice PCB graphic, tweak text
Add a nice citrus inspired PCB graphic for the bottom side of PlajTime v0.4
Other:
- board text added: "Main flash"
- board text removed: "2nd flash/RAM"

Commit message: Final Main PCB version
Parts:
- C44: renamed from C45; value TBD_H -> 270pF_H
- C45: renamed from C46; value TBD_H -> 270pF_H
- moved C21 0.69 mm to (41.8, 143.5), turned to 0 degrees
- renumbered C5 to C1, C11 to C10, C12 to C11, C13 to C12, C15 to C13, C1 to C15, C18 to C17, C19 to C18, C21 to C19, C4 to C2, C22 to C20, C24 to C21, C26 to C22, C25 to C24, C27 to C25, C28 to C26, C29 to C27, C30 to C28, C31 to C29, C6 to C3, C32 to C30, C33 to C31, C34 to C32, C35 to C33, C36 to C34, C37 to C35, C47 to C36, C39 to C37, C40 to C38, C41 to C39, C7 to C4, C42 to C40, C38 to C41, C43 to C42, C44 to C43, C2 to C5, C3 to C6, C8 to C7, C9 to C8, C10 to C9, J9 to J2, J2 to J3, J3 to J4, J4 to J5, J5 to J6, J8 to J7, J6 to J8, J7 to J9, L2 to L1, L1 to L2, R9 to R10, R10 to R11, R11 to R12, R12 to R2, R2 to R3, R3 to R4, R4 to R5, R5 to R6, R6 to R7, R7 to R8, R8 to R9, U9 to U1, U1 to U2, U2 to U4, U4 to U5, U5 to U6, U6 to U7, U7 to U8, U8 to U9
Routing:
- net GND: track 22.9 -> 22.1 mm, vias 83 -> 87
- net SDA: track 35.4 -> 34.9 mm
- net /CLK_OUT: track 27.3 -> 26.8 mm
