File: PCBs/plajtime-main/plajtime-main.kicad_sch (KiCad schematic)
At the start: 85 parts, among them J1 RP SWD, J2 RP USB, J3 Internal connector, J4 Display connector, J5 Extention connector, J6 Conn_Coaxial, J7 Battery Connector, J8 Nordic SWD, J9 Conn_Coaxial, U1 W25Q64JWUUIQ, U2 W25Q64JWBYIM, U3 TPS628438YKA, U4 MP2664, U5 RP2350A, U6 BMA456, U7 MAX17055, U8 RV-3028-C7, U9 nRF52833_QDxx, Y1 13MHz, Y2 32MHz

Commit message: main-pcb: Fix charger's power off mode, remove RTC
Parts:
- removed C28: 0.1uF, Capacitor_SMD:C_0201_0603Metric, symbol Device:C_Small
- removed R6, R7: 10k, Resistor_SMD:R_0201_0603Metric, symbol Device:R_Small
- removed U8: RV-3028-C7, Package_SON:MicroCrystal_C7_SON-8_1.5x3.2mm_P0.9mm, symbol Timer_RTC:RV-3028-C7
- added R13: 300k, symbol Device:R_Small
Connections:
- net CHARGER_INT: now also R13.2
- net CHG_VDD: now reaches C7.1, R1.1, U4.4 (VDD)
- net CHG_VDD: now also R13.1
Other:
- note added: "TODO: mby chose another it like works but too small hard to solder..."
- note added: "TODO: split to usb + i2c"

Commit message: PCB_main: Add 32.768kHz crystal, Split AUX and USB, retrace changes
Parts:
- removed J3: Internal connector, Library:CONN12_505066-1222_179x87_MOL, symbol Connector_Generic_MountingPin:Conn_02x06_Top_Bottom_MountingPin
- added C46, C47: TBD, Capacitor_SMD:C_0201_0603Metric, symbol Device:C_Small
- added J10: Internal connector, Library:5050660822, symbol Connector_Generic_MountingPin:Conn_02x04_Odd_Even_MountingPin
- added J11: USB, Library:CONN_505066-0622_MOL, symbol Connector_Generic_MountingPin:Conn_02x03_Odd_Even_MountingPin
- added Y3: 32.768kHz Crystal, Crystal:Crystal_SMD_MicroCrystal_CM9V-T1A-2Pin_1.6x1.0mm, symbol Device:Crystal
- R13: footprint (none) -> Resistor_SMD:R_0201_0603Metric
Connections:
- net FREEPIN is gone; now on net SDA: U9.5 (AIN3/P0.05)
- net RTC_INT is gone; now on net CHARGER_INT: U9.17 (P0.20)
- net +3V: now also J10.1 (Pin_1)
- net +5V: now also J11.1 (Pin_1), J11.3 (Pin_3)
- net CHARGER_INT: no longer U9.7 (P0.11)
- net GND: now also C46.2, C47.2, J10.2 (Pin_2), J10.7 (Pin_7), J10.MP (MountPin), J11.2 (Pin_2), J11.5 (Pin_5), J11.MP (MountPin)
- net GPU_INT: now also U9.7 (P0.11); no longer U9.4 (AIN2/P0.04)
- net RP_SCL: now also J10.3 (Pin_3)
- net RP_SDA: now also J10.5 (Pin_5)
- net SCL: now also U9.4 (AIN2/P0.04); no longer U9.2 (XL1/P0.00)
- net SDA: no longer U9.3 (XL2/P0.01)
- net SLIDER_INT: now also J10.6 (Pin_6)
- net USB_D+: now also J11.6 (Pin_6)
- net USB_D-: now also J11.4 (Pin_4)
- net VIC_INT: now also J10.4 (Pin_4)
- net VSYS: now also J10.8 (Pin_8)
- net CLK_OUT: no longer names the net of U5.37 (GPIO25)
- new net: C47.1, U9.3 (XL2/P0.01), Y3.1
- new net: C46.1, U9.2 (XL1/P0.00), Y3.2
- no-connect marks 14 -> 15
Other:
- note removed: "TODO: split to usb + i2c"
