File: PCBs/plajtime-main/plajtime-main.kicad_sch (KiCad schematic)
At the start: 86 parts, among them J1 RP SWD, J10 Internal connector, J11 USB, J2 RP USB, J4 Display connector, J5 Extention connector, J6 Conn_Coaxial, J7 Battery Connector, J8 Nordic SWD, J9 Conn_Coaxial, U1 W25Q64JWUUIQ, U2 W25Q64JWBYIM, U3 TPS628438YKA, U4 MP2664, U5 RP2350A, U6 BMA456, U7 MAX17055, U9 nRF52833_QDxx, Y1 13MHz, Y2 32MHz, Y3 32.768kHz Crystal

Commit message: Some fixes after v0.4
Connections:
- net GAUGE_INT: now also U9.7 (P0.11); no longer U9.6 (P1.09)
- net GPU_INT: now also U9.6 (P1.09); no longer U9.7 (P0.11)
Changed lines of the file:
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@@
 	(wire
 		(pts
-			(xy 372.11 182.88) (xy 361.95 182.88)
+			(xy 372.11 106.68) (xy 361.95 106.68)
 		)
 		(stroke
@@
 	)
 	(label "GAUGE_INT"
-		(at 372.11 182.88 180)
+		(at 372.11 106.68 180)
 		(effects
 			(font
@@
 	(global_label "GPU_INT"
 		(shape input)
-		(at 361.95 106.68 0)
+		(at 361.95 182.88 0)
 		(fields_autoplaced yes)
 		(effects
@@
 		)
 		(property "Intersheetrefs" "${INTERSHEET_REFS}"
-			(at 372.6762 106.68 0)
+			(at 372.6762 182.88 0)
 			(hide yes)
 			(show_name no)

Commit message: main-pcb: Fix Nordic USB (DECUSB), Improve I2C and RTC crystal routing
Also added labels for some nets, done basic board cleanup
Connections:
- net +3V: no longer C35.1, U9.11 (DECUSB)
- net RP_USB_D+: now reaches J2.2 (Pin_2), U5.52 (USB_DP)
- net RP_USB_D-: now reaches J2.3 (Pin_3), U5.51 (USB_DM)
- net NRF_XL2: now reaches C47.1, U9.3 (XL2/P0.01), Y3.1
- net NRF_XL1: now reaches C46.1, U9.2 (XL1/P0.00), Y3.2
- net RP_SWDCLK: now reaches J1.2 (Pin_2), U5.24 (SWCLK)
- net RP_SWDIO: now reaches J1.3 (Pin_3), U5.25 (SWDIO)
- net NRF_SWDRST: now reaches J8.1 (Pin_1), U9.16 (P0.18/~{RESET})
- net NRF_SWDCLK: now reaches J8.2 (Pin_2), U9.19 (SWDIO)
- net NRF_SWDIO: now reaches J8.3 (Pin_3), U9.20 (SWDCLK)
- new net NRF_DECUSB: C35.1, U9.11 (DECUSB)

Commit message: main-pcb: Fix charger shutdown properly
The previous fix used VDD (internal charger voltage), which was
not allowed. This fix uses the battery directly instead, to create
a pull-up on the INT pin. Additionally, a resistor is needed between
the sensing pin and the charger INT pin, because the nRF was pulling
it too hard, exceeding the minimum pin threshold. Therefore,
the resistor values should be calculated with this in mind.
Parts:
- added R14: TBD, Resistor_SMD:R_0201_0603Metric, symbol Device:R_Small
- R13: value 300k -> TBD
- Y1: value 13MHz -> 32MHz
Connections:
- net +BATT: now also R13.1
- net CHARGER_INT: now also R14.1; no longer R13.2, U4.3 (INT)
- net CHG_VDD: no longer R13.1
- new net: R13.2, R14.2, U4.3 (INT)
Changed lines of the file:
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@@
 	)
 	(junction
-		(at 68.58 224.79)
+		(at 64.77 217.17)
 		(diameter 0)
 		(color 0 0 0 0)
@@
 	(wire
 		(pts
-			(xy 68.58 224.79) (xy 83.82 224.79)
-		)
-		(stroke
-			(width 0)
-			(type default)
-		)
-	)
-	(wire
-		(pts
 			(xy 288.29 262.89) (xy 288.29 264.16)
 		)
@@
 	(wire
 		(pts
+			(xy 71.12 224.79) (xy 85.09 224.79)
+		)
+		(stroke
+			(width 0)
+			(type default)
+		)
+	)
+	(wire
+		(pts
 			(xy 48.26 43.18) (xy 40.64 43.18)
 		)
@@
 	(wire
 		(pts
-			(xy 68.58 220.98) (xy 68.58 224.79)
+			(xy 66.04 217.17) (xy 64.77 217.17)
 		)
 		(stroke
@@
 	(wire
 		(pts
-			(xy 68.58 215.9) (xy 68.58 214.63)
-		)
-		(stroke
-			(width 0)
-			(type default)
-		)
-	)
-	(wire
-		(pts
 			(xy 271.78 53.34) (xy 285.75 53.34)
 		)
@@
 	(wire
 		(pts
-			(xy 64.77 224.79) (xy 68.58 224.79)
+			(xy 72.39 217.17) (xy 71.12 217.17)
+		)
+		(stroke
+			(width 0)
+			(type default)
+		)
+	)
+	(wire
+		(pts
+			(xy 64.77 224.79) (xy 66.04 224.79)
 		)
 		(stroke
@@
 	(wire
 		(pts
-			(xy 68.58 214.63) (xy 77.47 214.63)
-		)
-		(stroke
-			(width 0)
-			(type default)
-		)
-	)
-	(wire
-		(pts
 			(xy 238.76 252.73) (xy 224.79 252.73)
 		)
@@
 		)
 	)
-	(label "CHG_VDD"
-		(at 77.47 214.63 180)
-		(effects
-			(font
-				(size 1.27 1.27)
-			)
-			(justify right bottom)
-		)
-	)
 	(label "CHARGER_INT"
-		(at 83.82 224.79 180)
+		(at 85.09 224.79 180)
 		(effects
 			(font
@@
 	)
 	(symbol
+		(lib_id "power:+BATT")
+		(at 72.39 217.17 0)
+		(unit 1)
+		(body_style 1)
+		(exclude_from_sim no)
+		(in_bom yes)
+		(on_board yes)
+		(in_pos_files yes)
+		(dnp no)
+		(property "Reference" "#PWR045"
+			(at 72.39 220.98 0)
+			(hide yes)
+			(show_name no)
+			(do_not_autoplace no)
+			(effects
+				(font
+					(size 1.27 1.27)
+				)
+			)
+		)
+		(property "Value" "+BATT"
+			(at 72.39 213.106 0)
+			(show_name no)
+			(do_not_autoplace no)
+			(effects
+				(font
+					(size 1.27 1.27)
+				)
+			)
+		)
+		(property "Footprint" ""
+			(at 72.39 217.17 0)
+			(hide yes)
+			(show_name no)
+			(do_not_autoplace no)
+			(effects
+				(font
+					(size 1.27 1.27)
+				)
+			)
+		)
+		(property "Datasheet" ""
+			(at 72.39 217.17 0)
+			(hide yes)
+			(show_name no)
+			(do_not_autoplace no)
+			(effects
+				(font
+					(size 1.27 1.27)
+				)
+			)
+		)
+		(property "Description" "Power symbol creates a global label with name \"+BATT\""
+			(at 72.39 217.17 0)
+			(hide yes)
+			(show_name no)
+			(do_not_autoplace no)
+			(effects
+				(font
+					(size 1.27 1.27)
+				)
+			)
+		)
+		(pin "1"
+		)
+		(instances
+			(project "plajtime-main"
+				(path "/ac4646bc-7c34-427b-b5dc-6b33046171d8"
+					(reference "#PWR045")
+					(unit 1)
+				)
+			)
+		)
+	)
+	(symbol
 		(lib_id "Device:C_Small")
 		(at 275.59 137.16 270)
@@
 			)
 		)
-		(property "Value" "13MHz"
+		(property "Value" "32MHz"
 			(at 46.736 167.132 90)
 			(show_name no)
@@
 		)
 		(property "Value" "GND"
-			(at 77.47 209.804 0)
+			(at 80.518 208.534 0)
 			(show_name no)
 			(do_not_autoplace no)
@@
 	(symbol
 		(lib_id "Device:R_Small")
-		(at 68.58 218.44 0)
+		(at 68.58 217.17 270)
 		(unit 1)
 		(body_style 1)
@@
 		(in_pos_files yes)
 		(dnp no)
-		(fields_autoplaced yes)
 		(property "Reference" "R13"
-			(at 71.12 217.1699 0)
+			(at 67.056 219.202 90)
 			(show_name no)
 			(do_not_autoplace no)
@@
 			)
 		)
-		(property "Value" "300k"
-			(at 71.12 219.7099 0)
+		(property "Value" "TBD"
+			(at 66.548 215.392 90)
 			(show_name no)
 			(do_not_autoplace no)
@@
 		)
 		(property "Footprint" "Resistor_SMD:R_0201_0603Metric"
-			(at 68.58 218.44 0)
+			(at 68.58 217.17 0)
 			(hide yes)
 			(show_name no)
@@
 		)
 		(property "Datasheet" ""
-			(at 68.58 218.44 0)
+			(at 68.58 217.17 0)
 			(hide yes)
 			(show_name no)
@@
 		)
 		(property "Description" "Resistor, small symbol"
-			(at 68.58 218.44 0)
+			(at 68.58 217.17 0)
 			(hide yes)
 			(show_name no)
@@
 					(unit 1)
 				)
+			)
+		)
+	)
+	(symbol
+		(lib_id "Device:R_Small")
+		(at 68.58 224.79 270)
+		(unit 1)
+		(body_style 1)
+		(exclude_from_sim no)
+		(in_bom yes)
+		(on_board yes)
+		(in_pos_files yes)
+		(dnp no)
+		(property "Reference" "R14"
+			(at 67.056 226.822 90)
+			(show_name no)
+			(do_not_autoplace no)
+			(effects
+				(font
+					(size 1.016 1.016)
+				)
+				(justify left)
+			)
+		)
+		(property "Value" "TBD"
+			(at 66.548 223.012 90)
+			(show_name no)
+			(do_not_autoplace no)
+			(effects
+				(font
+					(size 1.27 1.27)
+				)
+				(justify left)
+			)
+		)
+		(property "Footprint" "Resistor_SMD:R_0201_0603Metric"
+			(at 68.58 224.79 0)
+			(hide yes)
+			(show_name no)
+			(do_not_autoplace no)
+			(effects
+				(font
+					(size 1.27 1.27)
+				)
+			)
+		)
+		(property "Datasheet" ""
+			(at 68.58 224.79 0)
+			(hide yes)
+			(show_name no)
+			(do_not_autoplace no)
+			(effects
+				(font
+					(size 1.27 1.27)
+				)
+			)
+		)
+		(property "Description" "Resistor, small symbol"
+			(at 68.58 224.79 0)
+			(hide yes)
+			(show_name no)
+			(do_not_autoplace no)
+			(effects
+				(font
+					(size 1.27 1.27)
+				)
+			)
+		)
+		(pin "2"
+		)
+		(pin "1"
+		)
+		(instances
+			(project "plajtime-main"
+				(path "/ac4646bc-7c34-427b-b5dc-6b33046171d8"
+					(reference "R14")
+					(unit 1)
+				)
