File: PCBs/plajtime-bat-fpcb/plajtime-bat-fpcb.kicad_sch (KiCad schematic)
At the start: 9 parts, among them J7 Battery Connector, Q1 Q_Dual_NMOS_S1G1D2S2G2D1D1D2, U1 BQ297xy

Commit message: Done with battery FPCB
Parts:
- BT1: footprint (none) -> Library:Battery
- C1: footprint (none) -> Capacitor_SMD:C_0201_0603Metric
- Q1: footprint (none) -> Library:DFN1010B-6
- R1, R2, R3: footprint (none) -> Resistor_SMD:R_0201_0603Metric
- TH1: footprint C26706956 -> Resistor_SMD:R_0201_0603Metric
Changed lines of the file:
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@@
 			)
 		)
-		(property "Footprint" ""
+		(property "Footprint" "Library:Battery"
 			(at 64.77 58.166 90)
 			(effects
@@
 			)
 		)
-		(property "Footprint" ""
+		(property "Footprint" "Capacitor_SMD:C_0201_0603Metric"
 			(at 86.0552 67.31 0)
 			(effects
@@
 			)
 		)
-		(property "Footprint" ""
+		(property "Footprint" "Resistor_SMD:R_0201_0603Metric"
 			(at 156.972 57.15 90)
 			(effects
@@
 			)
 		)
-		(property "Footprint" ""
+		(property "Footprint" "Resistor_SMD:R_0201_0603Metric"
 			(at 83.312 52.07 90)
 			(effects
@@
 			)
 		)
-		(property "Footprint" ""
+		(property "Footprint" "Library:DFN1010B-6"
 			(at 146.05 73.66 0)
 			(effects
@@
 			)
 		)
-		(property "Footprint" "C26706956"
+		(property "Footprint" "Resistor_SMD:R_0201_0603Metric"
 			(at 59.69 57.15 0)
 			(effects
@@
 			)
 		)
-		(property "Footprint" ""
+		(property "Footprint" "Library:DFN1010B-6"
 			(at 135.89 73.66 0)
 			(effects
@@
 			)
 		)
-		(property "Footprint" ""
+		(property "Footprint" "Resistor_SMD:R_0201_0603Metric"
 			(at 36.322 58.42 90)
 			(effects
