File: PCBs/plajtime-bat-fpcb/plajtime-bat-fpcb.kicad_pcb (KiCad board)
At the start: 2 copper layers, 29.6 x 17.5 mm, 9 parts, among them J7 Battery Connector, Q1 Q_Dual_NMOS_S1G1D2S2G2D1D1D2, U1 BQ297xy

Commit message: Added stiffener for BAT FPCB
Other:
- board text added: "Pi stiffener T=0.2mm"
Changed lines of the file:
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@@
 		(39 "User.1" user)
 		(41 "User.2" user)
-		(43 "User.3" user)
-		(45 "User.4" user)
+		(43 "User.3" front "F.Stiffener")
+		(45 "User.4" back "B.Stiffener")
 	)
 	(setup
@@
 		(layer "Edge.Cuts")
 	)
+	(gr_arc
+		(start 85.540217 56.671898)
+		(mid 85.82306 56.789055)
+		(end 85.940217 57.071898)
+		(stroke
+			(width 0.1)
+			(type default)
+		)
+		(layer "User.3")
+	)
+	(gr_arc
+		(start 83.140217 57.071897)
+		(mid 83.257374 56.789055)
+		(end 83.540216 56.671898)
+		(stroke
+			(width 0.1)
+			(type default)
+		)
+		(layer "User.3")
+	)
+	(gr_line
+		(start 85.540217 60.671881)
+		(end 83.540216 60.67188)
+		(stroke
+			(width 0.1)
+			(type default)
+		)
+		(layer "User.3")
+	)
+	(gr_arc
+		(start 85.940216 60.271882)
+		(mid 85.823059 60.554724)
+		(end 85.540217 60.671881)
+		(stroke
+			(width 0.1)
+			(type default)
+		)
+		(layer "User.3")
+	)
+	(gr_line
+		(start 83.140216 60.27188)
+		(end 83.140216 57.0719)
+		(stroke
+			(width 0.1)
+			(type default)
+		)
+		(layer "User.3")
+	)
+	(gr_arc
+		(start 83.540216 60.67188)
+		(mid 83.257373 60.554724)
+		(end 83.140216 60.27188)
+		(stroke
+			(width 0.1)
+			(type default)
+		)
+		(layer "User.3")
+	)
+	(gr_line
+		(start 83.540216 56.671898)
+		(end 85.540217 56.671898)
+		(stroke
+			(width 0.1)
+			(type default)
+		)
+		(layer "User.3")
+	)
+	(gr_line
+		(start 85.940201 57.071898)
+		(end 85.940216 60.271882)
+		(stroke
+			(width 0.1)
+			(type default)
+		)
+		(layer "User.3")
+	)
 	(gr_line
 		(start 62.774898 74.171898)
@@
 	)
 	(gr_line
+		(start 56.726599 74.171902)
+		(end 67.79929 74.171902)
+		(stroke
+			(width 0.1)
+			(type default)
+		)
+		(layer "User.4")
+	)
+	(gr_arc
+		(start 68.79929 73.171193)
+		(mid 68.506646 73.878753)
+		(end 67.79929 74.171902)
+		(stroke
+			(width 0.1)
+			(type default)
+		)
+		(layer "User.4")
+	)
+	(gr_arc
+		(start 56.326598 71.171904)
+		(mid 56.443756 70.88906)
+		(end 56.726599 70.771902)
+		(stroke
+			(width 0.1)
+			(type default)
+		)
+		(layer "User.4")
+	)
+	(gr_line
+		(start 67.79831 70.771902)
+		(end 56.726599 70.771902)
+		(stroke
+			(width 0.1)
+			(type default)
+		)
+		(layer "User.4")
+	)
+	(gr_line
+		(start 56.326598 71.171904)
+		(end 56.326598 73.771899)
+		(stroke
+			(width 0.1)
+			(type default)
+		)
+		(layer "User.4")
+	)
+	(gr_arc
+		(start 67.79831 70.771902)
+		(mid 68.504731 71.064101)
+		(end 68.798323 71.769944)
+		(stroke
+			(width 0.1)
+			(type default)
+		)
+		(layer "User.4")
+	)
+	(gr_line
 		(start 84.540217 60.671898)
 		(end 84.540217 56.671898)
@@
 		)
 		(layer "User.4")
+	)
+	(gr_arc
+		(start 56.726599 74.171902)
+		(mid 56.443756 74.054744)
+		(end 56.326598 73.771899)
+		(stroke
+			(width 0.1)
+			(type default)
+		)
+		(layer "User.4")
+	)
+	(gr_line
+		(start 68.798296 71.769944)
+		(end 68.79929 73.171193)
+		(stroke
+			(width 0.1)
+			(type default)
+		)
+		(layer "User.4")
+	)
+	(gr_text "Pi stiffener\nT=0.2mm"
+		(at 80.65 56.09 0)
+		(layer "User.3")
+		(effects
+			(font
+				(size 1 1)
+				(thickness 0.15)
+			)
+			(justify left bottom)
+		)
+	)
+	(gr_text "Pi stiffener\nT=0.2mm"
+		(at 58.9 70.19 0)
+		(layer "User.4")
+		(effects
+			(font
+				(size 1 1)
+				(thickness 0.15)
+			)
+			(justify left bottom)
+		)
 	)
 	(dimension
@@
 			(keep_text_aligned yes)
 		)
-		(gr_text "17,5"
+		(gr_text "17.5"
 			(at 52.45 65.421898 90)
 			(layer "Cmts.User")
@@
 			(keep_text_aligned yes)
 		)
-		(gr_text "29,6136"
+		(gr_text "29.6136"
 			(at 71.13341 77.65 0)
 			(layer "Cmts.User")
