File: PCBs/plajtime-bat-fpcb/plajtime-bat-fpcb.kicad_pcb (KiCad board)
At the start: 2 copper layers, 29.6 x 17.5 mm, 9 parts, among them J7 Battery Connector, Q1 Q_Dual_NMOS_S1G1D2S2G2D1D1D2, U1 BQ297xy

Commit message: Add 3D models for AUX board and connectors
Parts:
- Q1: value Q_Dual_NMOS_S1G1D2S2G2D1D1D2 -> NX7002BKXBZ
Changed lines of the file:
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@@
 			)
 		)
-		(property "Value" "Q_Dual_NMOS_S1G1D2S2G2D1D1D2"
+		(property "Value" "NX7002BKXBZ"
 			(at -11.9 -14.3 270)
 			(unlocked yes)
@@
 			)
 		)
-		(property "Datasheet" "~"
+		(property "Datasheet" "https://www.lcsc.com/datasheet/C551613.pdf"
 			(at 0 0 270)
 			(unlocked yes)
@@
 		)
 		(embedded_fonts no)
+		(model "${KICAD9_3DMODEL_DIR}/Package_DFN_QFN.3dshapes/DFN-6-1EP_1.2x1.2mm_P0.4mm_EP0.3x0.94mm.step"
+			(offset
+				(xyz 0 0 0)
+			)
+			(scale
+				(xyz 0.9 0.9 0.9)
+			)
+			(rotate
+				(xyz -0 -0 -90)
+			)
+		)
 	)
 	(footprint "Capacitor_SMD:C_0201_0603Metric"
@@
 		)
 		(embedded_fonts no)
+		(model "${KIPRJMOD}/3D_models/5050700622.stp"
+			(offset
+				(xyz 0 0 0)
+			)
+			(scale
+				(xyz 1 1 1)
+			)
+			(rotate
+				(xyz 0 0 0)
+			)
+		)
 	)
 	(gr_poly
