File: PCBs/plajtime-aux/plajtime-aux.kicad_pcb (KiCad board)
At the start: 2 copper layers, 50.7 x 23.5 mm, 21 parts, among them J1 Slider, J2 USB, J3 Internal connector, J4 LRA, U1 USBLC6-2P6, U2 IQS7222B, U3 DA7280

Commit message: Done with AUX board
Parts:
- J4: footprint Connector_PinHeader_1.00mm:PinHeader_1x02_P1.00mm_Vertical -> Library:PinHeader_1x02_P1.00mm_Vertical
- moved J4 0.10 mm to (74.7, 80.0)
Routing:
- net GND: track 19.6 -> 22.5 mm, vias 31 -> 32
Other:
- board text added: "Pi stiffener T=0.2mm"
