File: PCBs/plajtime-aux/plajtime-aux.kicad_sch (KiCad schematic)
At the start: 0 parts

Commit message: feat: Add new KiCad project for battery flexible PCB, updating main, auxiliary, and 3D models.
Parts:
- added C1: 0.1uF, symbol Device:C
- added C2, C4, C6: 100pF, symbol Device:C
- added C3, C5: 2.2uF, symbol Device:C
- added C7: 4.7uF, symbol Device:C
- added C8: 0.1uF, symbol Device:C_Small
- added D1: D_shottky, Diode_SMD:D_SOD-123, symbol Device:D_Schottky_Small
- added J1: Slider, Library:TouchSlider-5_26.2x4.2mm, symbol Connector:Conn_01x05_Pin
- added J2: USB, symbol Connector:Conn_01x04_Pin
- added J3: Internal connector, Library:CONN12_505066-1222_179x87_MOL, symbol Connector_Generic_MountingPin:Conn_02x06_Top_Bottom_MountingPin
- added J4: LRA, symbol Connector:Conn_01x02_Pin
- added R1, R2, R3, R4, R5: 470, symbol Device:R_Small
- added U1: USBLC6-2P6, Package_TO_SOT_SMD:SOT-666, symbol Power_Protection:USBLC6-2P6
- added U2: IQS7222B, Package_DFN_QFN:QFN-20-1EP_3x3mm_P0.4mm_EP1.65x1.65mm, symbol Library:IQS7222B
- added U3: DA7280, symbol Library:DA7280
Connections:
- new net: J2.2 (Pin_2), U1.3 (I/O2)
- new net: J2.3 (Pin_3), U1.1 (I/O1)
- new net: D1.2 (A), J2.4 (Pin_4)
- new net: J1.1 (Pin_1), R1.1
- new net: R1.2, U2.5 (CR/CTx0)
- new net: C4.1, C5.1, U2.2 (VREGD)
- new net: C1.1, U2.20 (MCLR/GPIO6)
- new net: C2.1, C3.1, U2.4 (VREGA)
- new net: R4.2, U2.6 (CR/CTx1)
- new net: R2.2, U2.7 (CR/CTx2)
- new net: R5.2, U2.8 (CR/CTx3)
- new net: R3.2, U2.9 (CR/CTx4)
- new net: J4.1 (Pin_1), U3.8 (OUTN)
- new net: J4.2 (Pin_2), U3.5 (OUTP)
- new net: J1.2 (Pin_2), R4.1
- new net: J1.3 (Pin_3), R2.1
- new net: J1.4 (Pin_4), R5.1
- new net: J1.5 (Pin_5), R3.1
- new net: C8.2, U3.6 (GND_1)
- new net +3V: C6.1, C7.1, J3.1 (Pin_1), U2.1 (VDD), U3.9 (VDDIO)
- new net +5V: D1.1 (K), J3.10 (Pin_10), J3.9 (Pin_9), U1.5 (VBUS)
- new net GND: C1.2, C2.2, C3.2, C4.2, C5.2, C6.2, C7.2, J2.1 (Pin_1), J3.2 (Pin_2), J3.3 (Pin_3), J3.MP (MountPin), U1.2 (GND), U2.14 (CTx9/GPIO0), U2.15 (CTx10/GPIO3), U2.16 (CTx11/GPIO4), U2.3 (VSS), U3.7 (GND_2)
- new net RP_SCL: J3.4 (Pin_4), U2.18 (SCL/GPIO2), U3.11 (SCL)
- new net RP_SDA: J3.5 (Pin_5), U2.19 (SDA/GPIO1), U3.10 (SDA)
- new net SLIDER_INT: J3.6 (Pin_6), U2.17 (RDY/GPIO5)
- new net USB_D+: J3.11 (Pin_11), U1.6 (I/O1)
- new net USB_D-: J3.12 (Pin_12), U1.4 (I/O2)
- new net VBUS: C8.1, J3.7 (Pin_7), U3.4 (VDD)
- new net VIC_INT: J3.8 (Pin_8), U3.12 (nIRQ)
- no-connect marks 0 -> 7

Commit message: Almost done AUX Board
Parts:
- C1, C2, C3, C4, C5, C6, C8: footprint (none) -> Capacitor_SMD:C_0201_0603Metric
- C7: footprint (none) -> Capacitor_SMD:C_0402_1005Metric
- D1: footprint Diode_SMD:D_SOD-123 -> Diode_SMD:D_0402_1005Metric
- J1: footprint Library:TouchSlider-5_26.2x4.2mm -> Library:TouchSlider-5_25.0248x4.2mm
- J2: footprint (none) -> Library:PinHeader_1x04_P2.54mm_Vertical
- J3: footprint Library:CONN12_505066-1222_179x87_MOL -> Library:5050701222
- J4: footprint (none) -> Connector_PinHeader_1.00mm:PinHeader_1x02_P1.00mm_Vertical
- R1, R2, R3, R4, R5: footprint (none) -> Resistor_SMD:R_0201_0603Metric
- U1: footprint Package_TO_SOT_SMD:SOT-666 -> Library:PESD3V3L5UF115
- U3: footprint (none) -> Library:BGA12C40P3X4_135X175X58
Connections:
- net +3V: now also U3.B3 (VDDIO); no longer U3.9 (VDDIO)
- net GND: now also C8.2, U2.21 (EP), U3.C3 (GND_2), U3.D3 (GND_1); no longer U3.7 (GND_2)
- net RP_SCL: now also U3.A2 (SCL); no longer U3.11 (SCL)
- net RP_SDA: now also U3.A3 (SDA); no longer U3.10 (SDA)
- net VBUS: now also U3.D1 (VDD); no longer U3.4 (VDD)
- net VIC_INT: now also U3.A1 (nIRQ); no longer U3.12 (nIRQ)
- net D-: now reaches J2.2 (Pin_2), U1.3 (I/O2)
- net D+: now reaches J2.3 (Pin_3), U1.1 (I/O1)
- net at J4.1 (Pin_1): now also U3.C2 (OUTN); no longer U3.8 (OUTN)
- net at J4.2 (Pin_2): now also U3.D2 (OUTP); no longer U3.5 (OUTP)
Changed lines of the file:
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@@
 	)
 	(junction
+		(at 195.58 100.33)
+		(diameter 0)
+		(color 0 0 0 0)
+	)
+	(junction
 		(at 153.67 82.55)
 		(diameter 0)
@@
 		)
 	)
+	(label "D-"
+		(at 50.8 45.72 0)
+		(effects
+			(font
+				(size 1.27 1.27)
+			)
+			(justify left bottom)
+		)
+	)
 	(label "SLIDER_INT"
 		(at 39.37 115.57 0)
@@
 		)
 	)
+	(label "D+"
+		(at 50.8 43.18 0)
+		(effects
+			(font
+				(size 1.27 1.27)
+			)
+			(justify left bottom)
+		)
+	)
 	(label "SLIDER_INT"
 		(at 160.02 46.99 0)
@@
 			)
 		)
-		(property "Footprint" ""
+		(property "Footprint" "Library:PinHeader_1x04_P2.54mm_Vertical"
 			(at 45.72 45.72 0)
 			(effects
@@
 			)
 		)
-		(property "Footprint" ""
+		(property "Footprint" "Resistor_SMD:R_0201_0603Metric"
 			(at 40.64 82.55 0)
 			(effects
@@
 			)
 		)
-		(property "Datasheet" ""
+		(property "Datasheet" "https://www.azoteq.com/images/stories/pdf/iqs7222b_datasheet.pdf"
 			(at 67.31 102.87 0)
 			(effects
@@
 			)
 		)
-		(property "Footprint" "Diode_SMD:D_SOD-123"
+		(property "Footprint" "Diode_SMD:D_0402_1005Metric"
 			(at 57.15 36.83 90)
 			(effects
@@
 			)
 		)
-		(property "Footprint" ""
+		(property "Footprint" "Connector_PinHeader_1.00mm:PinHeader_1x02_P1.00mm_Vertical"
 			(at 246.38 107.95 0)
 			(effects
@@
 			)
 		)
-		(property "Footprint" ""
+		(property "Footprint" "Resistor_SMD:R_0201_0603Metric"
 			(at 45.72 85.09 0)
 			(effects
@@
 			)
 		)
-		(property "Footprint" ""
+		(property "Footprint" "Capacitor_SMD:C_0201_0603Metric"
 			(at 87.3252 102.87 0)
 			(effects
@@
 			)
 		)
-		(property "Footprint" "Library:TouchSlider-5_26.2x4.2mm"
+		(property "Footprint" "Library:TouchSlider-5_25.0248x4.2mm"
 			(at 29.21 87.63 0)
 			(effects
@@
 			)
 		)
-		(property "Footprint" "Library:CONN12_505066-1222_179x87_MOL"
+		(property "Footprint" "Library:5050701222"
 			(at 176.53 39.37 0)
 			(effects
@@
 			)
 		)
-		(property "Footprint" ""
+		(property "Footprint" "Capacitor_SMD:C_0201_0603Metric"
 			(at 127.9652 97.79 0)
 			(effects
@@
 			)
 		)
-		(property "Footprint" ""
+		(property "Footprint" "Capacitor_SMD:C_0201_0603Metric"
 			(at 113.9952 97.79 0)
 			(effects
@@
 			)
 		)
-		(property "Footprint" ""
+		(property "Footprint" "Capacitor_SMD:C_0201_0603Metric"
 			(at 101.2952 102.87 0)
 			(effects
@@
 	)
 	(symbol
+		(lib_id "power:GND")
+		(at 195.58 100.33 0)
+		(unit 1)
+		(exclude_from_sim no)
+		(in_bom yes)
+		(on_board yes)
+		(dnp no)
+		(property "Reference" "#PWR021"
+			(at 195.58 106.68 0)
+			(effects
+				(font
+					(size 1.27 1.27)
+				)
+				(hide yes)
+			)
+		)
+		(property "Value" "GND"
+			(at 195.58 104.902 0)
+			(effects
+				(font
+					(size 1.27 1.27)
+				)
+			)
+		)
+		(property "Footprint" ""
+			(at 195.58 100.33 0)
+			(effects
+				(font
+					(size 1.27 1.27)
+				)
+				(hide yes)
+			)
+		)
+		(property "Datasheet" ""
+			(at 195.58 100.33 0)
+			(effects
+				(font
+					(size 1.27 1.27)
+				)
+				(hide yes)
+			)
+		)
+		(property "Description" "Power symbol creates a global label with name \"GND\" , ground"
+			(at 195.58 100.33 0)
+			(effects
+				(font
+					(size 1.27 1.27)
+				)
+				(hide yes)
+			)
+		)
+		(pin "1"
+		)
+		(instances
+			(project "plajtime-aux"
+				(path "/4927e521-23d4-4b4c-83b6-f3b54e580c82"
+					(reference "#PWR021")
+					(unit 1)
+				)
+			)
+		)
+	)
+	(symbol
 		(lib_id "power:+3.3V")
 		(at 163.83 34.29 0)
@@
 			)
 		)
-		(property "Footprint" ""
+		(property "Footprint" "Resistor_SMD:R_0201_0603Metric"
 			(at 40.64 87.63 0)
 			(effects
@@
 			)
 		)
-		(property "Footprint" ""
+		(property "Footprint" "Resistor_SMD:R_0201_0603Metric"
 			(at 45.72 90.17 0)
 			(effects
@@
 			)
 		)
-		(property "Footprint" ""
+		(property "Footprint" "Capacitor_SMD:C_0201_0603Metric"
 			(at 195.58 96.52 0)
 			(effects
@@
 			)
 		)
-		(property "Footprint" ""
+		(property "Footprint" "Capacitor_SMD:C_0201_0603Metric"
 			(at 140.6652 92.71 0)
 			(effects
@@
 			)
 		)
-		(property "Footprint" ""
+		(property "Footprint" "Resistor_SMD:R_0201_0603Metric"
 			(at 40.64 92.71 0)
 			(effects
@@
 			)
 		)
-		(property "Footprint" ""
+		(property "Footprint" "Library:BGA12C40P3X4_135X175X58"
 			(at 220.98 111.76 0)
 			(effects
@@
 			)
 		)
-		(pin "4"
+		(pin "A1"
 		)
-		(pin "6"
+		(pin "C2"
 		)
-		(pin "12"
+		(pin "B1"
 		)
-		(pin "8"
+		(pin "C1"
 		)
-		(pin "2"
+		(pin "C3"
 		)
-		(pin "3"
+		(pin "B3"
 		)
-		(pin "9"
+		(pin "D3"
 		)
-		(pin "7"
+		(pin "D1"
 		)
-		(pin "5"
+		(pin "D2"
 		)
-		(pin "11"
+		(pin "A2"
 		)
-		(pin "10"
+		(pin "A3"
 		)
-		(pin "1"
+		(pin "B2"
 		)
 		(instances
@@
 			)
 		)
-		(property "Footprint" ""
+		(property "Footprint" "Capacitor_SMD:C_0402_1005Metric"
 			(at 154.6352 92.71 0)
 			(effects
@@
 			)
 		)
-		(property "Footprint" "Package_TO_SOT_SMD:SOT-666"
+		(property "Footprint" "Library:PESD3V3L5UF115"
 			(at 65.786 49.911 0)
 			(effects
@@
 			)
 		)
-		(property "Footprint" ""
+		(property "Footprint" "Capacitor_SMD:C_0201_0603Metric"
 			(at 47.9552 132.08 0)
 			(effects

Commit message: Done with AUX board
Parts:
- J4: footprint Connector_PinHeader_1.00mm:PinHeader_1x02_P1.00mm_Vertical -> Library:PinHeader_1x02_P1.00mm_Vertical
Changed lines of the file:
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@@
 			)
 		)
-		(property "Footprint" "Connector_PinHeader_1.00mm:PinHeader_1x02_P1.00mm_Vertical"
+		(property "Footprint" "Library:PinHeader_1x02_P1.00mm_Vertical"
 			(at 246.38 107.95 0)
 			(effects
